Commit message: feat(mola): minor update for texture

File: stonefish_ws/src/MBARI/MOLA_AUV/mola_auv_sim/urdf/mola_auv.urdf.xacro (robot description, xacro)
@@ -45,7 +45,7 @@
         <geometry>
           <mesh
-            filename="package://mola_auv_sim/data/mola_auv/mesh/rviz/mola_auv_lightL.stl" scale="1.0 1.0 1.0"/>
-        </geometry>
-        <material name="light"/>
+            filename="package://mola_auv_sim/data/mola_auv/mesh/rviz/mola_auv_lightL.obj" scale="1.0 1.0 1.0"/>
+        </geometry>
+        <!-- <material name="light"/> -->
       </visual>
     </link>
@@ -57,7 +57,7 @@
         <geometry>
           <mesh
-            filename="package://mola_auv_sim/data/mola_auv/mesh/rviz/mola_auv_lightR.stl" scale="1.0 1.0 1.0"/>
-        </geometry>
-        <material name="light"/>
+            filename="package://mola_auv_sim/data/mola_auv/mesh/rviz/mola_auv_lightR.obj" scale="1.0 1.0 1.0"/>
+        </geometry>
+        <!-- <material name="light"/> -->
       </visual>
     </link>
