Commit message: feat(mola): wip propellers.
TODO: TF publisher for joint state from stonefish topics

File: stonefish_ws/src/MBARI/MOLA_AUV/mola_auv_sim/urdf/materials.xacro (robot description, xacro)
@@ -11,5 +11,8 @@
     </material>
     <material name="glass">
-        <color rgba="1.0 1.0 1.0 1"/>
+        <color rgba="1.0 1.0 1.0 0.5"/>
+    </material>
+    <material name="yellow">
+        <color rgba="0.898 0.769 0.145"/>
     </material>
     <material name="base">

File: stonefish_ws/src/MBARI/MOLA_AUV/mola_auv_sim/urdf/mola_auv.urdf.xacro (robot description, xacro)
@@ -62,4 +62,164 @@
       </visual>
     </link>
+    <!-- PROPELLER LFU -->
+    <link name="mola_auv_propLFU">
+      <visual>
+        <origin
+          xyz="0 0 0"
+          rpy="0 0 0" />
+        <geometry>
+          <mesh
+            filename="package://mola_auv_sim/data/mola_auv/mesh/rviz/ccw.stl" scale="1.17 1.17 1.17"/>
+        </geometry>
+        <material name="yellow"/>
+      </visual>
+    </link>
+    <joint name="base_propLFU" type="continuous">
+      <origin rpy="0.0 -${45*pi/180} -${135*pi/180}" xyz="0.3 -0.182 -0.105"/>
+      <parent link="mola_auv_base" />
+      <child link="mola_auv_propLFU" />
+			<axis xyz="1.0 0.0 0.0"/>
+			<limit effort="1.0" velocity="1.0"/>
+    </joint>
+    <!-- PROPELLER LFD -->
+    <link name="mola_auv_propLFD">
+      <visual>
+        <origin
+          xyz="0 0 0"
+          rpy="0 0 0" />
+        <geometry>
+          <mesh
+            filename="package://mola_auv_sim/data/mola_auv/mesh/rviz/cw.stl" scale="1.17 1.17 1.17"/>
+        </geometry>
+        <material name="yellow"/>
+      </visual>
+    </link>
+    <joint name="base_propLFD" type="continuous">
+      <origin rpy="0.0 ${45*pi/180} -${135*pi/180}" xyz="0.3 -0.182 0.105"/>
+      <parent link="mola_auv_base" />
+      <child link="mola_auv_propLFD" />
+			<axis xyz="1.0 0.0 0.0"/>
+			<limit effort="1.0" velocity="1.0"/>
+    </joint>
+   <!-- PROPELLER RFU -->
+    <link name="mola_auv_propRFU">
+      <visual>
+        <origin
+          xyz="0 0 0"
+          rpy="0 0 0" />
+        <geometry>
+          <mesh
+            filename="package://mola_auv_sim/data/mola_auv/mesh/rviz/cw.stl" scale="1.17 1.17 1.17"/>
+        </geometry>
+        <material name="yellow"/>
+      </visual>
+    </link>
+    <joint name="base_propRFU" type="continuous">
+      <origin rpy="0.0 -${45*pi/180} ${135*pi/180}" xyz="0.3 0.182 -0.105"/>
+      <parent link="mola_auv_base" />
+      <child link="mola_auv_propRFU" />
+			<axis xyz="1.0 0.0 0.0"/>
+			<limit effort="1.0" velocity="1.0"/>
+    </joint>
+   <!-- PROPELLER RFD -->
+    <link name="mola_auv_propRFD">
+      <visual>
+        <origin
+          xyz="0 0 0"
+          rpy="0 0 0" />
+        <geometry>
+          <mesh
+            filename="package://mola_auv_sim/data/mola_auv/mesh/rviz/ccw.stl" scale="1.17 1.17 1.17"/>
+        </geometry>
+        <material name="yellow"/>
+      </visual>
+    </link>
+    <joint name="base_propRFD" type="continuous">
+      <origin rpy="0.0 ${45*pi/180} ${135*pi/180}" xyz="0.3 0.182 0.105"/>
+      <parent link="mola_auv_base" />
+      <child link="mola_auv_propRFD" />
+			<axis xyz="1.0 0.0 0.0"/>
+			<limit effort="1.0" velocity="1.0"/>
+    </joint>
+    <!-- PROPELLER LBU -->
+    <link name="mola_auv_propLBU">
+      <visual>
+        <origin
+          xyz="0 0 0"
+          rpy="0 0 0" />
+        <geometry>
+          <mesh
+            filename="package://mola_auv_sim/data/mola_auv/mesh/rviz/ccw.stl" scale="1.17 1.17 1.17"/>
+        </geometry>
+        <material name="yellow"/>
+      </visual>
+    </link>
+    <joint name="base_propLBU" type="continuous">
+      <origin rpy="0.0 ${45*pi/180} ${135*pi/180}" xyz="-0.3 -0.182 -0.105"/>
+      <parent link="mola_auv_base" />
+      <child link="mola_auv_propLBU" />
+			<axis xyz="1.0 0.0 0.0"/>
+			<limit effort="1.0" velocity="1.0"/>
+    </joint>
+   <!-- PROPELLER LBD -->
+    <link name="mola_auv_propLBD">
+      <visual>
+        <origin
+          xyz="0 0 0"
+          rpy="0 0 0" />
+        <geometry>
+          <mesh
+            filename="package://mola_auv_sim/data/mola_auv/mesh/rviz/cw.stl" scale="1.17 1.17 1.17"/>
+        </geometry>
+        <material name="yellow"/>
+      </visual>
+    </link>
+    <joint name="base_propLBD" type="continuous">
+      <origin rpy="0.0 -${45*pi/180} ${135*pi/180}" xyz="-0.3 -0.182 0.105"/>
+      <parent link="mola_auv_base" />
+      <child link="mola_auv_propLBD" />
+			<axis xyz="1.0 0.0 0.0"/>
+			<limit effort="1.0" velocity="1.0"/>
+    </joint>
+    <!-- PROPELLER RBU -->
+    <link name="mola_auv_propRBU">
+      <visual>
+        <origin
+          xyz="0 0 0"
+          rpy="0 0 0" />
+        <geometry>
+          <mesh
+            filename="package://mola_auv_sim/data/mola_auv/mesh/rviz/cw.stl" scale="1.17 1.17 1.17"/>
+        </geometry>
+        <material name="yellow"/>
+      </visual>
+    </link>
+    <joint name="base_propRBU" type="continuous">
+      <origin rpy="0.0 ${45*pi/180} -${135*pi/180}" xyz="-0.3 0.182 -0.105"/>
+      <parent link="mola_auv_base" />
+      <child link="mola_auv_propRBU" />
+			<axis xyz="1.0 0.0 0.0"/>
+			<limit effort="1.0" velocity="1.0"/>
+    </joint>
+    <!-- PROPELLER RBD -->
+    <link name="mola_auv_propRBD">
+      <visual>
+        <origin
+          xyz="0 0 0"
+          rpy="0 0 0" />
+        <geometry>
+          <mesh
+            filename="package://mola_auv_sim/data/mola_auv/mesh/rviz/ccw.stl" scale="1.17 1.17 1.17"/>
+        </geometry>
+        <material name="yellow"/>
+      </visual>
+    </link>
+    <joint name="base_propRBD" type="continuous">
+      <origin rpy="0.0 -${45*pi/180} -${135*pi/180}" xyz="-0.3 0.182 0.105"/>
+      <parent link="mola_auv_base" />
+      <child link="mola_auv_propRBD" />
+			<axis xyz="1.0 0.0 0.0"/>
+			<limit effort="1.0" velocity="1.0"/>
+    </joint>
     <joint name="base_frame" type="fixed">
       <origin rpy="0 0 0" xyz="0 0 0"/>

Commit message: feat(mola): further clean up and fixed thrusters

File: stonefish_ws/src/MBARI/MOLA_AUV/mola_auv_sim/urdf/materials.xacro (robot description, xacro)
@@ -14,5 +14,5 @@
     </material>
     <material name="yellow">
-        <color rgba="0.898 0.769 0.145"/>
+        <color rgba="0.898 0.769 0.145 1.0"/>
     </material>
     <material name="base">

File: stonefish_ws/src/MBARI/MOLA_AUV/mola_auv_sim/urdf/mola_auv.urdf.xacro (robot description, xacro)
@@ -75,5 +75,5 @@
       </visual>
     </link>
-    <joint name="base_propLFU" type="continuous">
+    <!-- <joint name="base_propLFU" type="continuous">
       <origin rpy="0.0 -${45*pi/180} -${135*pi/180}" xyz="0.3 -0.182 -0.105"/>
       <parent link="mola_auv_base" />
@@ -81,4 +81,9 @@
 			<axis xyz="1.0 0.0 0.0"/>
 			<limit effort="1.0" velocity="1.0"/>
+    </joint> -->
+    <joint name="base_propLFU" type="fixed">
+      <origin rpy="0.0 -${45*pi/180} -${135*pi/180}" xyz="0.3 -0.182 -0.105"/>
+      <parent link="mola_auv_base" />
+      <child link="mola_auv_propLFU" />
     </joint>
     <!-- PROPELLER LFD -->
@@ -95,5 +100,5 @@
       </visual>
     </link>
-    <joint name="base_propLFD" type="continuous">
+    <!-- <joint name="base_propLFD" type="continuous">
       <origin rpy="0.0 ${45*pi/180} -${135*pi/180}" xyz="0.3 -0.182 0.105"/>
       <parent link="mola_auv_base" />
@@ -101,4 +106,9 @@
 			<axis xyz="1.0 0.0 0.0"/>
 			<limit effort="1.0" velocity="1.0"/>
+    </joint> -->
+    <joint name="base_propLFD" type="fixed">
+      <origin rpy="0.0 ${45*pi/180} -${135*pi/180}" xyz="0.3 -0.182 0.105"/>
+      <parent link="mola_auv_base" />
+      <child link="mola_auv_propLFD" />
     </joint>
    <!-- PROPELLER RFU -->
@@ -115,5 +125,5 @@
       </visual>
     </link>
-    <joint name="base_propRFU" type="continuous">
+    <!-- <joint name="base_propRFU" type="continuous">
       <origin rpy="0.0 -${45*pi/180} ${135*pi/180}" xyz="0.3 0.182 -0.105"/>
       <parent link="mola_auv_base" />
@@ -121,4 +131,9 @@
 			<axis xyz="1.0 0.0 0.0"/>
 			<limit effort="1.0" velocity="1.0"/>
+    </joint> -->
+    <joint name="base_propRFU" type="fixed">
+      <origin rpy="0.0 -${45*pi/180} ${135*pi/180}" xyz="0.3 0.182 -0.105"/>
+      <parent link="mola_auv_base" />
+      <child link="mola_auv_propRFU" />
     </joint>
    <!-- PROPELLER RFD -->
@@ -135,5 +150,5 @@
       </visual>
     </link>
-    <joint name="base_propRFD" type="continuous">
+    <!-- <joint name="base_propRFD" type="continuous">
       <origin rpy="0.0 ${45*pi/180} ${135*pi/180}" xyz="0.3 0.182 0.105"/>
       <parent link="mola_auv_base" />
@@ -141,4 +156,9 @@
 			<axis xyz="1.0 0.0 0.0"/>
 			<limit effort="1.0" velocity="1.0"/>
+    </joint> -->
+    <joint name="base_propRFD" type="fixed">
+      <origin rpy="0.0 ${45*pi/180} ${135*pi/180}" xyz="0.3 0.182 0.105"/>
+      <parent link="mola_auv_base" />
+      <child link="mola_auv_propRFD" />
     </joint>
     <!-- PROPELLER LBU -->
@@ -155,5 +175,5 @@
       </visual>
     </link>
-    <joint name="base_propLBU" type="continuous">
+    <!-- <joint name="base_propLBU" type="continuous">
       <origin rpy="0.0 ${45*pi/180} ${135*pi/180}" xyz="-0.3 -0.182 -0.105"/>
       <parent link="mola_auv_base" />
@@ -161,4 +181,9 @@
 			<axis xyz="1.0 0.0 0.0"/>
 			<limit effort="1.0" velocity="1.0"/>
+    </joint> -->
+    <joint name="base_propLBU" type="fixed">
+      <origin rpy="0.0 ${45*pi/180} ${135*pi/180}" xyz="-0.3 -0.182 -0.105"/>
+      <parent link="mola_auv_base" />
+      <child link="mola_auv_propLBU" />
     </joint>
    <!-- PROPELLER LBD -->
@@ -175,5 +200,5 @@
       </visual>
     </link>
-    <joint name="base_propLBD" type="continuous">
+    <!-- <joint name="base_propLBD" type="continuous">
       <origin rpy="0.0 -${45*pi/180} ${135*pi/180}" xyz="-0.3 -0.182 0.105"/>
       <parent link="mola_auv_base" />
@@ -181,4 +206,9 @@
 			<axis xyz="1.0 0.0 0.0"/>
 			<limit effort="1.0" velocity="1.0"/>
+    </joint> -->
+    <joint name="base_propLBD" type="fixed">
+      <origin rpy="0.0 -${45*pi/180} ${135*pi/180}" xyz="-0.3 -0.182 0.105"/>
+      <parent link="mola_auv_base" />
+      <child link="mola_auv_propLBD" />
     </joint>
     <!-- PROPELLER RBU -->
@@ -195,5 +225,5 @@
       </visual>
     </link>
-    <joint name="base_propRBU" type="continuous">
+    <!-- <joint name="base_propRBU" type="continuous">
       <origin rpy="0.0 ${45*pi/180} -${135*pi/180}" xyz="-0.3 0.182 -0.105"/>
       <parent link="mola_auv_base" />
@@ -201,4 +231,9 @@
 			<axis xyz="1.0 0.0 0.0"/>
 			<limit effort="1.0" velocity="1.0"/>
+    </joint> -->
+    <joint name="base_propRBU" type="fixed">
+      <origin rpy="0.0 ${45*pi/180} -${135*pi/180}" xyz="-0.3 0.182 -0.105"/>
+      <parent link="mola_auv_base" />
+      <child link="mola_auv_propRBU" />
     </joint>
     <!-- PROPELLER RBD -->
@@ -215,5 +250,5 @@
       </visual>
     </link>
-    <joint name="base_propRBD" type="continuous">
+    <!-- <joint name="base_propRBD" type="continuous">
       <origin rpy="0.0 -${45*pi/180} -${135*pi/180}" xyz="-0.3 0.182 0.105"/>
       <parent link="mola_auv_base" />
@@ -221,4 +256,9 @@
 			<axis xyz="1.0 0.0 0.0"/>
 			<limit effort="1.0" velocity="1.0"/>
+    </joint> -->
+    <joint name="base_propRBD" type="fixed">
+      <origin rpy="0.0 -${45*pi/180} -${135*pi/180}" xyz="-0.3 0.182 0.105"/>
+      <parent link="mola_auv_base" />
+      <child link="mola_auv_propRBD" />
     </joint>
     <joint name="base_frame" type="fixed">
